File: PCB_files/Eagle_v0.2/easy_bee_counter.sch (EAGLE design)
At the start: 123 parts, among them Q6 60V/32A/35mΩ, Q7 60V/32A/35mΩ

Commit message: Converted Logo to library part Added vias to be solded bridged for jumpers to bypass the SIP resistors. Rerouted the board, realigned many of the parts.
Parts:
- added U$44: BEE_LOGO, owen_desktop:BEE_LOGO
- C7: value 1uF -> 0.1uF
- J1: value (none) -> S_5V
- J3: value (none) -> S_LOAD
- J4: value (none) -> S_I2C
- R11, R12, R2, R5, R6, R7: value (none) -> 100KΩ
- U$34, U$35, U$36, U$37: value RPACK-BUSSED-9 -> 22Ω
- U1, U2, U3, U4, U5, U6: value (none) -> 74*165
- U7: value (none) -> R78E3.3-1.0; device SparkFun-IC-Power:V_REG_78XXSINK -> SparkFun-IC-Power:R-78E5.0-1.0
Connections:
- removed net N$44: U$45.MOSI

Commit message: Reworked connections to 74*165s to put the sense pins in a better order for the board layout.
Parts:
- removed U$100, U$101, U$102, U$103, U$104, U$105, U$106, U$107, U$108, U$109, U$110, U$111, U$112, U$113, U$114, U$115, U$68, U$69, U$70, U$71, U$72, U$73, U$74, U$75, U$76, U$77, U$78, U$79, U$80, U$81, U$82, U$83, U$84, U$85, U$86, U$87, U$88, U$89, U$90, U$91, U$92, U$93, U$94, U$95, U$96, U$97, U$98, U$99: QRE1113_, QRE1113:QRE1113_
- added SERVO1, SERVO2, SERVO3, SERVO4, SERVO5: (no value), pinhead:PINHD-1X3
- added U01I, U01O, U02I, U02O, U03I, U03O, U04I, U04O, U05I, U05O, U06I, U06O, U07I, U07O, U08I, U08O, U09I, U09O, U10I, U10O, U11I, U11O, U12I, U12O, U13I, U13O, U14I, U14O, U15I, U15O, U16I, U16O, U17I, U17O, U18I, U18O, U19I, U19O, U20I, U20O, U21I, U21O, U22I, U22O, U23I, U23O, U24I, U24O: QRE1113_QRE1113_, easy_bee_counter:QRE1113_QRE1113_
Connections:
- net N$21 renamed PWR_13-24
- net N$63 renamed PWR_1-12
- removed net N$101: R12.4, U$112.E, U6.C
- removed net N$102: R12.5, U$113.E, U6.D
- removed net N$105: R11.5, U$105.E, U5.D
- removed net N$108: R12.8, U$108.E, U6.G
- removed net N$109: R12.9, U$109.E, U6.H
- removed net N$112: R11.9, U$101.E, U5.H
- removed net N$117: R11.7, U$103.E, U5.F
- removed net N$12: R5.9, U$77.E, U2.H
- removed net N$131: R7.5, U$97.E, U4.D
- removed net N$135: R7.9, U$93.E, U4.H
- removed net N$140: R7.7, U$95.E, U4.F
- removed net N$141: R7.3, U$99.E, U4.B
- removed net N$15: R6.3, U$90.E, U3.A
- removed net N$16: R6.2, U$91.E, U3.B
- removed net N$17: R6.4, U$88.E, U3.C
- removed net N$18: R12.6, U$110.E, U6.E
- removed net N$19: R6.5, U$89.E, U3.D
- removed net N$20: R6.8, U$84.E, U3.G
- removed net N$22: R6.9, U$85.E, U3.H
- removed net N$23: R6.6, U$86.E, U3.E
- removed net N$24: R6.7, U$87.E, U3.F
- removed net N$25: R5.4, U$80.E, U2.C
- removed net N$26: R5.5, U$81.E, U2.D
- removed net N$27: R5.8, U$76.E, U2.G
- removed net N$29: R5.6, U$78.E, U2.E
- removed net N$30: R12.3, U$114.E, U6.A
- removed net N$32: R5.7, U$79.E, U2.F
- removed net N$33: R5.3, U$83.E, U2.B
- removed net N$34: R7.4, U$96.E, U4.C
- removed net N$35: R5.2, U$82.E, U2.A
- removed net N$36: R2.7, U$72.E, U1.C
- removed net N$37: R2.6, U$73.E, U1.D
- removed net N$38: R2.5, U$68.E, U1.G
- removed net N$39: R2.4, U$69.E, U1.H
- removed net N$40: R2.2, U$70.E, U1.E
- removed net N$41: R2.3, U$71.E, U1.F
- removed net N$42: R2.8, U$75.E, U1.B
- removed net N$43: R2.9, U$74.E, U1.A
- removed net N$58: R12.7, U$111.E, U6.F
- removed net N$62: R7.8, U$92.E, U4.G
- removed net N$65: R7.6, U$94.E, U4.E
- removed net N$68: R7.2, U$98.E, U4.A
- removed net N$74: R11.3, U$107.E, U5.B
- removed net N$87: R12.2, U$115.E, U6.B
- removed net N$89: R11.4, U$104.E, U5.C
- removed net N$91: R11.8, U$100.E, U5.G
- removed net N$93: R11.6, U$102.E, U5.E
- removed net N$97: R11.2, U$106.E, U5.A
- new net SNS01I: R12.3, U01I.E, U6.F
- new net SNS01O: R12.2, U01O.E, U6.E
- new net SNS02I: R12.5, U02I.E, U6.H
- new net SNS02O: R12.4, U02O.E, U6.G
- new net SNS03I: R12.7, U03I.E, U6.C
- new net SNS03O: R12.6, U03O.E, U6.D
- new net SNS04I: R12.9, U04I.E, U6.A
- new net SNS04O: R12.8, U04O.E, U6.B
- new net SNS05I: R11.3, U05I.E, U5.F
- new net SNS05O: R11.2, U05O.E, U5.E
- new net SNS06I: R11.5, U06I.E, U5.H
- new net SNS06O: R11.4, U06O.E, U5.G
- new net SNS07I: R11.7, U07I.E, U5.C
- new net SNS07O: R11.6, U07O.E, U5.D
- new net SNS08I: R11.9, U08I.E, U5.A
- new net SNS08O: R11.8, U08O.E, U5.B
- new net SNS09I: R7.3, U09I.E, U4.F
- new net SNS09O: R7.2, U09O.E, U4.E
- new net SNS10I: R7.5, U10I.E, U4.H
- new net SNS10O: R7.4, U10O.E, U4.G
- new net SNS11I: R7.7, U11I.E, U4.C
- new net SNS11O: R7.6, U11O.E, U4.D
- new net SNS12I: R7.9, U12I.E, U4.A
- new net SNS12O: R7.8, U12O.E, U4.B
- new net SNS13I: R6.3, U13I.E, U3.F
- new net SNS13O: R6.2, U13O.E, U3.E
- new net SNS14I: R6.5, U14I.E, U3.H
- new net SNS14O: R6.4, U14O.E, U3.G
- new net SNS15I: R6.7, U15I.E, U3.C
- new net SNS15O: R6.6, U15O.E, U3.D
- new net SNS16I: R6.9, U3.A
- new net SNS16O: R6.8, U3.B
- new net SNS17I: R5.3, U17I.E, U2.F
- new net SNS17O: R5.2, U17O.E, U2.E
- new net SNS18I: R5.5, U18I.E, U2.H
- new net SNS18O: R5.4, U18O.E, U2.G
- new net SNS19I: R5.7, U19I.E, U2.C
- new net SNS19O: R5.6, U19O.E, U2.D
- new net SNS20I: R5.9, U2.A
- new net SNS20O: R5.8, U2.B
- new net SNS21I: R2.3, U1.F, U21I.E
- new net SNS21O: R2.2, U1.E, U21O.E
- new net SNS22I: R2.5, U1.H, U22I.E
- new net SNS22O: R2.4, U1.G, U22O.E
- new net SNS23I: R2.7, U1.C
- new net SNS23O: R2.6, U1.D
- new net SNS24I: R2.9, U1.A
- new net SNS24O: R2.8, U1.B
- new net SRVO1: MS2.GPIOA0, SERVO1.3, U$45.A1
- new net SRVO2: MS2.GPIOA1, SERVO2.3, U$45.A2
- new net SRVO3: MS2.GPIOA2, SERVO3.3, U$45.A3
- new net SRVO4: MS2.GPIO13, SERVO4.3, U$45.D13
- new net SRVO5: MS2.GPIO12, SERVO5.3, U$45.D9
- net 10_CATHODE: now also U10O.K; no longer U$97.K
- net 11_CATHODE: now also U11O.K; no longer U$95.K
- net 12_CATHODE: now also U12O.K; no longer U$93.K
- net 13_CATHODE: now also U13O.K; no longer U$91.K
- net 14_CATHODE: now also U14O.K; no longer U$89.K
- net 15_CATHODE: now also U15O.K; no longer U$87.K
- net 16_CATHODE: now also U16O.K; no longer U$85.K
- net 17_CATHODE: now also U17O.K; no longer U$83.K
- net 18_CATHODE: now also U18O.K; no longer U$81.K
- net 19_CATHODE: now also U19O.K; no longer U$79.K
- net 1_CATHODE: now also U01O.K; no longer U$115.K
- net 20_CATHODE: now also U20O.K; no longer U$77.K
- net 21_CATHODE: now also U21O.K; no longer U$75.K
- net 22_CATHODE: now also U22O.K; no longer U$73.K
- net 23_CATHODE: now also U23O.K; no longer U$71.K
- net 24_CATHODE: now also U24O.K; no longer U$69.K
- net 2_CATHODE: now also U02O.K; no longer U$113.K
- net 3.3V: now also U01I.A, U01I.C, U01O.C, U02I.A, U02I.C, U02O.C, U03I.A, U03I.C, U03O.C, U04I.A, U04I.C, U04O.C, U05I.A, U05I.C, U05O.C, U06I.A, U06I.C, U06O.C, U07I.A, U07I.C, U07O.C, U08I.A, U08I.C, U08O.C, U09I.A, U09I.C, U09O.C, U10I.A, U10I.C, U10O.C, U11I.A, U11I.C, U11O.C, U12I.A, U12I.C, U12O.C, U13I.A, U13I.C, U13O.C, U14I.A, U14I.C, U14O.C, U15I.A, U15I.C, U15O.C, U16I.A, U16I.C, U16O.C, U17I.A, U17I.C, U17O.C, U18I.A, U18I.C, U18O.C, U19I.A, U19I.C, U19O.C, U20I.A, U20I.C, U20O.C, U21I.A, U21I.C, U21O.C, U22I.A, U22I.C, U22O.C, U23I.A, U23I.C, U23O.C, U24I.A, U24I.C, U24O.C; no longer U$100.A, U$100.C, U$101.C, U$102.A, U$102.C, U$103.C, U$104.A, U$104.C, U$105.C, U$106.A, U$106.C, U$107.C, U$108.A, U$108.C, U$109.C, U$110.A, U$110.C, U$111.C, U$112.A, U$112.C, U$113.C, U$114.A, U$114.C, U$115.C, U$68.A, U$68.C, U$69.C, U$70.A, U$70.C, U$71.C, U$72.A, U$72.C, U$73.C, U$74.A, U$74.C, U$75.C, U$76.A, U$76.C, U$77.C, U$78.A, U$78.C, U$79.C, U$80.A, U$80.C, U$81.C, U$82.A, U$82.C, U$83.C, U$84.A, U$84.C, U$85.C, U$86.A, U$86.C, U$87.C, U$88.A, U$88.C, U$89.C, U$90.A, U$90.C, U$91.C, U$92.A, U$92.C, U$93.C, U$94.A, U$94.C, U$95.C, U$96.A, U$96.C, U$97.C, U$98.A, U$98.C, U$99.C
- net 3_CATHODE: now also U03O.K; no longer U$111.K
- net 4_CATHODE: now also U04O.K; no longer U$109.K
- net 5V: now also SERVO1.2, SERVO2.2, SERVO3.2, SERVO4.2, SERVO5.2
- net 5_CATHODE: now also U05O.K; no longer U$107.K
- net 6_CATHODE: now also U06O.K; no longer U$105.K
- net 7_CATHODE: now also U07O.K; no longer U$103.K
- net 8_CATHODE: now also U08O.K; no longer U$101.K
- net 9_CATHODE: now also U09O.K; no longer U$99.K
- net GND: now also SERVO1.1, SERVO2.1, SERVO3.1, SERVO4.1, SERVO5.1
- net N$1: now also U11I.K, U11O.A; no longer U$94.K, U$95.A
- net N$10: now also U07I.K, U07O.A; no longer U$102.K, U$103.A
- net N$11: now also U03I.K, U03O.A; no longer U$110.K, U$111.A
- net N$13: now also U02I.K, U02O.A; no longer U$112.K, U$113.A
- net N$14: now also U01I.K, U01O.A; no longer U$114.K, U$115.A
- net N$2: now also U12I.K, U12O.A; no longer U$92.K, U$93.A
- net N$3: now also U10I.K, U10O.A; no longer U$96.K, U$97.A
- net N$4: now also U09I.K, U09O.A; no longer U$98.K, U$99.A
- net N$45: now also U24I.K, U24O.A; no longer U$68.K, U$69.A
- net N$46: now also U23I.K, U23O.A; no longer U$70.K, U$71.A
- net N$47: now also U22I.K, U22O.A; no longer U$72.K, U$73.A
- net N$48: now also U21I.K, U21O.A; no longer U$74.K, U$75.A
- net N$49: now also U17I.K, U17O.A; no longer U$82.K, U$83.A
- net N$5: now also U05I.K, U05O.A; no longer U$106.K, U$107.A
- net N$50: now also U18I.K, U18O.A; no longer U$80.K, U$81.A
- net N$51: now also U20I.K, U20O.A; no longer U$76.K, U$77.A
- net N$52: now also U19I.K, U19O.A; no longer U$78.K, U$79.A
- net N$53: now also U16I.K, U16O.A; no longer U$84.K, U$85.A
- net N$54: now also U15I.K, U15O.A; no longer U$86.K, U$87.A
- net N$55: now also U14I.K, U14O.A; no longer U$88.K, U$89.A
- net N$56: now also U13I.K, U13O.A; no longer U$90.K, U$91.A
- net N$6: now also U06I.K, U06O.A; no longer U$104.K, U$105.A
- net N$7: now also U08I.K, U08O.A; no longer U$100.K, U$101.A
- net N$8: now also U04I.K, U04O.A; no longer U$108.K, U$109.A
Other:
- moved on the sheet: C1, C2, C3, C4, C5, U1, U2, U3, U4, U5

Commit message: Finalized all connections on schematic (missed some sensors last commit). Fully routed board using new component names and new pinouts for SIP packs.
Connections:
- removed net N$28: U3.QH, U4.SER
- new net SER5: U1.QH, U2.SER
- net SER3: now also U3.QH, U4.SER; no longer U2.QH, U3.SER
- net SER4: now also U2.QH, U3.SER; no longer U1.QH, U2.SER
- net SNS16I: now also U16I.E
- net SNS16O: now also U16O.E
- net SNS20I: now also U20I.E
- net SNS20O: now also U20O.E
- net SNS23I: now also U23I.E
- net SNS23O: now also U23O.E
- net SNS24I: now also U24I.E
- net SNS24O: now also U24O.E
- net SRVO1: now also U$45.A(0); no longer U$45.A1
- net SRVO2: now also U$45.A1; no longer U$45.A2
- net SRVO3: now also U$45.A2; no longer U$45.A3
Changed lines of the file:
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@@
 <drawing>
 <settings>
-<setting alwaysvectorfont="no"/>
+<setting alwaysvectorfont="yes"/>
 <setting keepoldvectorfont="yes"/>
 <setting verticaltext="up"/>
@@
 <segment>
 <wire x1="-50.8" y1="756.92" x2="-50.8" y2="871.22" width="0.1524" layer="91"/>
-<wire x1="-50.8" y1="871.22" x2="-175.26" y2="871.22" width="0.1524" layer="91"/>
+<wire x1="-50.8" y1="871.22" x2="-91.44" y2="871.22" width="0.1524" layer="91"/>
 <pinref part="R6" gate="G$1" pin="8"/>
 <label x="-142.24" y="871.22" size="1.778" layer="95"/>
 <pinref part="U3" gate="U1" pin="B"/>
+<wire x1="-91.44" y1="871.22" x2="-175.26" y2="871.22" width="0.1524" layer="91"/>
 <wire x1="-50.8" y1="756.92" x2="-27.94" y2="756.92" width="0.1524" layer="91"/>
+<pinref part="U16O" gate="G$1" pin="E"/>
+<wire x1="-91.44" y1="878.84" x2="-91.44" y2="871.22" width="0.1524" layer="91"/>
+<junction x="-91.44" y="871.22"/>
 </segment>
 </net>
@@
 <segment>
 <wire x1="-48.26" y1="873.76" x2="-48.26" y2="754.38" width="0.1524" layer="91"/>
-<wire x1="-175.26" y1="873.76" x2="-48.26" y2="873.76" width="0.1524" layer="91"/>
+<wire x1="-175.26" y1="873.76" x2="-109.22" y2="873.76" width="0.1524" layer="91"/>
 <pinref part="R6" gate="G$1" pin="9"/>
 <label x="-142.24" y="873.76" size="1.778" layer="95"/>
 <pinref part="U3" gate="U1" pin="A"/>
+<wire x1="-109.22" y1="873.76" x2="-48.26" y2="873.76" width="0.1524" layer="91"/>
 <wire x1="-48.26" y1="754.38" x2="-27.94" y2="754.38" width="0.1524" layer="91"/>
+<pinref part="U16I" gate="G$1" pin="E"/>
+<wire x1="-109.22" y1="878.84" x2="-109.22" y2="873.76" width="0.1524" layer="91"/>
+<junction x="-109.22" y="873.76"/>
 </segment>
 </net>
@@
 <segment>
 <wire x1="-48.26" y1="919.48" x2="-48.26" y2="1038.86" width="0.1524" layer="91"/>
-<wire x1="-48.26" y1="1038.86" x2="-172.72" y2="1038.86" width="0.1524" layer="91"/>
+<wire x1="-48.26" y1="1038.86" x2="-91.44" y2="1038.86" width="0.1524" layer="91"/>
 <pinref part="R5" gate="G$1" pin="8"/>
 <label x="-142.24" y="1038.86" size="1.778" layer="95"/>
 <pinref part="U2" gate="U1" pin="B"/>
+<wire x1="-91.44" y1="1038.86" x2="-172.72" y2="1038.86" width="0.1524" layer="91"/>
 <wire x1="-48.26" y1="919.48" x2="-30.48" y2="919.48" width="0.1524" layer="91"/>
+<pinref part="U20O" gate="G$1" pin="E"/>
+<wire x1="-91.44" y1="1046.48" x2="-91.44" y2="1038.86" width="0.1524" layer="91"/>
+<junction x="-91.44" y="1038.86"/>
 </segment>
 </net>
@@
 <net name="SNS24O" class="0">
 <segment>
-<wire x1="-144.78" y1="1188.72" x2="-50.8" y2="1188.72" width="0.1524" layer="91"/>
+<wire x1="-144.78" y1="1188.72" x2="-91.44" y2="1188.72" width="0.1524" layer="91"/>
+<wire x1="-91.44" y1="1188.72" x2="-50.8" y2="1188.72" width="0.1524" layer="91"/>
 <wire x1="-50.8" y1="1074.42" x2="-50.8" y2="1188.72" width="0.1524" layer="91"/>
 <pinref part="R2" gate="G$1" pin="8"/>
@@
 <pinref part="U1" gate="U1" pin="B"/>
 <wire x1="-50.8" y1="1074.42" x2="-30.48" y2="1074.42" width="0.1524" layer="91"/>
+<pinref part="U24O" gate="G$1" pin="E"/>
+<wire x1="-91.44" y1="1196.34" x2="-91.44" y2="1188.72" width="0.1524" layer="91"/>
+<junction x="-91.44" y="1188.72"/>
 </segment>
 </net>
 <net name="SNS23O" class="0">
 <segment>
-<wire x1="-152.4" y1="1155.7" x2="-55.88" y2="1155.7" width="0.1524" layer="91"/>
+<wire x1="-152.4" y1="1155.7" x2="-91.44" y2="1155.7" width="0.1524" layer="91"/>
+<wire x1="-91.44" y1="1155.7" x2="-55.88" y2="1155.7" width="0.1524" layer="91"/>
 <wire x1="-55.88" y1="1079.5" x2="-55.88" y2="1155.7" width="0.1524" layer="91"/>
 <pinref part="R2" gate="G$1" pin="6"/>
@@
 <pinref part="U1" gate="U1" pin="D"/>
 <wire x1="-55.88" y1="1079.5" x2="-30.48" y2="1079.5" width="0.1524" layer="91"/>
+<pinref part="U23O" gate="G$1" pin="E"/>
+<wire x1="-91.44" y1="1163.32" x2="-91.44" y2="1155.7" width="0.1524" layer="91"/>
+<junction x="-91.44" y="1155.7"/>
 </segment>
 </net>
@@
 <segment>
 <wire x1="-53.34" y1="1158.24" x2="-53.34" y2="1076.96" width="0.1524" layer="91"/>
-<wire x1="-53.34" y1="1158.24" x2="-149.86" y2="1158.24" width="0.1524" layer="91"/>
+<wire x1="-53.34" y1="1158.24" x2="-109.22" y2="1158.24" width="0.1524" layer="91"/>
 <pinref part="R2" gate="G$1" pin="7"/>
+<wire x1="-109.22" y1="1158.24" x2="-149.86" y2="1158.24" width="0.1524" layer="91"/>
 <wire x1="-170.18" y1="1178.56" x2="-149.86" y2="1178.56" width="0.1524" layer="91"/>
 <wire x1="-149.86" y1="1178.56" x2="-149.86" y2="1158.24" width="0.1524" layer="91"/>
@@
 <pinref part="U1" gate="U1" pin="C"/>
 <wire x1="-53.34" y1="1076.96" x2="-30.48" y2="1076.96" width="0.1524" layer="91"/>
+<pinref part="U23I" gate="G$1" pin="E"/>
+<wire x1="-109.22" y1="1163.32" x2="-109.22" y2="1158.24" width="0.1524" layer="91"/>
+<junction x="-109.22" y="1158.24"/>
 </segment>
 </net>
@@
 <segment>
 <wire x1="-45.72" y1="1041.4" x2="-45.72" y2="916.94" width="0.1524" layer="91"/>
-<wire x1="-45.72" y1="1041.4" x2="-172.72" y2="1041.4" width="0.1524" layer="91"/>
+<wire x1="-45.72" y1="1041.4" x2="-109.22" y2="1041.4" width="0.1524" layer="91"/>
 <pinref part="R5" gate="G$1" pin="9"/>
 <label x="-142.24" y="1041.4" size="1.778" layer="95"/>
 <pinref part="U2" gate="U1" pin="A"/>
+<wire x1="-109.22" y1="1041.4" x2="-172.72" y2="1041.4" width="0.1524" layer="91"/>
 <wire x1="-45.72" y1="916.94" x2="-30.48" y2="916.94" width="0.1524" layer="91"/>
+<pinref part="U20I" gate="G$1" pin="E"/>
+<wire x1="-109.22" y1="1046.48" x2="-109.22" y2="1041.4" width="0.1524" layer="91"/>
+<junction x="-109.22" y="1041.4"/>
 </segment>
 </net>
@@
 <segment>
 <wire x1="-48.26" y1="1191.26" x2="-48.26" y2="1071.88" width="0.1524" layer="91"/>
-<wire x1="-48.26" y1="1191.26" x2="-147.32" y2="1191.26" width="0.1524" layer="91"/>
+<wire x1="-48.26" y1="1191.26" x2="-109.22" y2="1191.26" width="0.1524" layer="91"/>
 <pinref part="R2" gate="G$1" pin="9"/>
+<wire x1="-109.22" y1="1191.26" x2="-147.32" y2="1191.26" width="0.1524" layer="91"/>
 <wire x1="-170.18" y1="1183.64" x2="-147.32" y2="1183.64" width="0.1524" layer="91"/>
 <wire x1="-147.32" y1="1183.64" x2="-147.32" y2="1191.26" width="0.1524" layer="91"/>
@@
 <pinref part="U1" gate="U1" pin="A"/>
 <wire x1="-48.26" y1="1071.88" x2="-30.48" y2="1071.88" width="0.1524" layer="91"/>
+<pinref part="U24I" gate="G$1" pin="E"/>
+<wire x1="-109.22" y1="1196.34" x2="-109.22" y2="1191.26" width="0.1524" layer="91"/>
+<junction x="-109.22" y="1191.26"/>
 </segment>
 </net>
@@
 <wire x1="5.08" y1="436.88" x2="-5.08" y2="436.88" width="0.1524" layer="91"/>
 <label x="5.08" y="274.32" size="1.778" layer="95"/>
+<label x="5.08" y="360.68" size="1.778" layer="95"/>
 </segment>
 </net>
@@
 <wire x1="-7.62" y1="591.82" x2="0" y2="591.82" width="0.1524" layer="91"/>
 <label x="2.54" y="449.58" size="1.778" layer="95"/>
+<label x="0" y="500.38" size="1.778" layer="95"/>
 </segment>
 </net>
-<net name="SER3" class="0">
+<net name="SER4" class="0">
 <segment>
 <pinref part="U3" gate="U1" pin="SER"/>
@@
 <pinref part="U2" gate="U1" pin="QH"/>
 <wire x1="2.54" y1="929.64" x2="-10.16" y2="929.64" width="0.1524" layer="91"/>
-<label x="5.08" y="769.62" size="1.778" layer="95"/>
+<label x="2.54" y="802.64" size="1.778" layer="95" rot="R90"/>
 </segment>
 </net>
-<net name="SER4" class="0">
+<net name="SER5" class="0">
 <segment>
 <pinref part="U2" gate="U1" pin="SER"/>
@@
 </segment>
 </net>
-<net name="N$28" class="0">
+<net name="SER3" class="0">
 <segment>
 <pinref part="U4" gate="U1" pin="SER"/>
@@
 <net name="SRVO3" class="0">
 <segment>
-<pinref part="U$45" gate="G$1" pin="A3"/>
-<wire x1="-246.38" y1="1049.02" x2="-254" y2="1049.02" width="0.1524" layer="91"/>
-<label x="-254" y="1049.02" size="1.778" layer="95"/>
-</segment>
-<segment>
 <pinref part="SERVO3" gate="A" pin="3"/>
 <wire x1="-347.98" y1="830.58" x2="-347.98" y2="807.72" width="0.1524" layer="91"/>
@@
 <label x="-200.66" y="985.52" size="1.778" layer="95"/>
 </segment>
-</net>
-<net name="SRVO2" class="0">
 <segment>
 <pinref part="U$45" gate="G$1" pin="A2"/>
@@
 <label x="-254" y="1051.56" size="1.778" layer="95"/>
 </segment>
+</net>
+<net name="SRVO2" class="0">
 <segment>
 <pinref part="MS2" gate="G$1" pin="GPIOA1"/>
@@
 <label x="-335.28" y="812.8" size="1.778" layer="95" rot="R90"/>
 </segment>
+<segment>
+<pinref part="U$45" gate="G$1" pin="A1"/>
+<wire x1="-246.38" y1="1054.1" x2="-254" y2="1054.1" width="0.1524" layer="91"/>
+<label x="-254" y="1054.1" size="1.778" layer="95"/>
+</segment>
 </net>
 <net name="SRVO4" class="0">
@@
 <net name="SRVO1" class="0">
 <segment>
-<pinref part="U$45" gate="G$1" pin="A1"/>
-<wire x1="-246.38" y1="1054.1" x2="-254" y2="1054.1" width="0.1524" layer="91"/>
-<label x="-254" y="1054.1" size="1.778" layer="95"/>
-</segment>
-<segment>
 <pinref part="MS2" gate="G$1" pin="GPIOA0"/>
 <wire x1="-210.82" y1="980.44" x2="-185.42" y2="980.44" width="0.1524" layer="91"/>
@@
 <label x="-322.58" y="812.8" size="1.778" layer="95" rot="R90"/>
 </segment>
+<segment>
+<pinref part="U$45" gate="G$1" pin="A(0)"/>
+<wire x1="-246.38" y1="1056.64" x2="-254" y2="1056.64" width="0.1524" layer="91"/>
+<label x="-254" y="1056.64" size="1.778" layer="95"/>
+</segment>
 </net>
